File: comm_v0p6/comm_v0p6.kicad_pcb (KiCad board)
At the start: 4 copper layers, 40 x 40 mm, 12 parts, among them J1 1x15 header, J2 1x15 socket, J4 2x2 socket, J5 2x2 socket, J6 2x2 socket, J7 2x2 socket, U1 ATmega328PB-M, Y1 20MHz

Commit message: prepare revision 3
Other:
- board text added: "+5V"
- board text added: "2024-07-29"
- board text added: "BOTTOM"
- board text added: "CIPO"
- board text added: "COPI"
- board text added: "CS0"
- board text added: "CS1"
- board text added: "CS2"
- board text added: "CS3"
- board text added: "CS4"
- board text added: "CS5"
- board text added: "CS6"
- board text added: "CS7"
- board text added: "EXT"
- board text added: "G4.1 Comm V0.6r3"
- board text added: "GND"
- board text added: "RST"
- board text added: "SCK"
- board text added: "https://reiserlab.github.io /Modular-LED-Display /G4"
- board text removed: "BOT"
- board text removed: "G4 Comm V0.6 Rev1"
