File: comm_v0p6/comm_v0p6.kicad_sch (KiCad schematic)
At the start: 12 parts, among them J1 1x15 header, J2 1x15 socket, J4 2x2 socket, J5 2x2 socket, J6 2x2 socket, J7 2x2 socket, U1 ATmega328PB-M, Y1 20MHz

Commit message: prepare revision 3
Parts:
- C3: LCSC PN C5137499 -> C66501
- J2: LCSC Alternative C2897397 -> (none); LCSC PN (none) -> C2897397
- J4, J5, J6, J7: LCSC Alternative C718234 -> (none); LCSC PN (none) -> C718234
- U1: LCSC PN C2651953 -> C2651951
Other:
- company: (none) -> Reiser Lab @ Janelia
- title: (none) -> G4.1 Comm Board
