File: panel-tester_arduino-uno/panel-tester_arduino-uno.kicad_sch (KiCad schematic)
At the start: 2 parts, among them J1 Conn_01x15_Female

Commit message: make tester ready for order
Connections:
- net CS1: now also J1.8 (Pin_8), XA1.D9; no longer J1.7 (Pin_7), XA1.D10 (D10_CS)
- net CIPO: now reaches XA1.D12
- net CIPO: now also J1.6 (Pin_6)
- net CS7: now reaches XA1.D3 (D3_INT1)
- net CS7: now also J1.14 (Pin_14)
- net CS6: now reaches XA1.D4
- net CS6: now also J1.13 (Pin_13)
- net CS5: now reaches XA1.D5
- net CS5: now also J1.12 (Pin_12)
- net CS4: now reaches XA1.D6
- net CS4: now also J1.11 (Pin_11)
- net CS3: now reaches XA1.D7
- net CS3: now also J1.10 (Pin_10)
- net CS2: now reaches XA1.D8
- net CS2: now also J1.9 (Pin_9)
- new net CS0: J1.7 (Pin_7), XA1.D10 (D10_CS)
Other:
- company: (none) -> MCN-NET for Reiser lab @ Janelia
- title: (none) -> G4 Panel Tester
